Commit message: Update with gripper stl; update roboreg end link to combined gripper / finger stl; add stl to urdf

File: plugins/server_roboreg/xarm7_standalone.urdf (robot description, URDF)
Before this commit: robot UF_ROBOT, 18 links, 17 joints
Links:
- link link_eef: geometry collision mesh filename=assets/xarm_gripper_fixed_open.stl; visual mesh filename=assets/xarm_gripper_fixed_open.stl
